File: 16ChannelServoControllerDaughterboardDesign/16ChannelServoControllerDaughterboardDesign.kicad_pcb (KiCad board)
At the start: 2 copper layers, 100 x 53.5 mm, 19 parts, among them J1 DaughterBoard, J2 8ServoConnectSym, J3 8ServoConnectSym, J4 Conn_01x03, J6 Screw_Terminal_01x02, Q1 BSS138, Q2 BSS138, U1 PCA9685PW

Commit message: created _latest gerber sets and added digikey boms. Also did some project cleanup WedMay82024
Routing:
- net GND: vias 4 -> 142
Other:
- board text added: "GP21"
