File: myBaseBoardDesignv1/myBaseBoardDesignv1.kicad_pcb (KiCad board)
At the start: 2 copper layers, 100 x 100 mm, 17 parts, among them J1 BaseBoard, J2 Barrel_Jack_Switch, J3 Conn_01x02, J4 Screw_Terminal_01x02, Q2 DMP6180SK3, SW1 SW_SPDT, U1 ESP32-S3-DevKitC

Commit message: two more projects ..HeartLEDTHT & TPA3122D2_Amplifier
Routing:
- net VIN: track 135.5 -> 138.2 mm, vias 2 -> 4
- net GP18: track 41.4 -> 42.2 mm
- net GP17: track 41.5 -> 42.2 mm
Changed lines of the file:
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@@
 		(tags "Through hole pin header THT 1x02 2.54mm single row")
 		(property "Reference" "J3"
-			(at 2.75 3.525 270)
+			(at 2.75 3.525 -90)
 			(layer "F.SilkS")
 			(effects
@@
 		)
 		(property "Value" "Conn_01x02"
-			(at 0 4.87 270)
+			(at 0 4.87 -90)
 			(layer "F.Fab")
 			(effects
@@
 		)
 		(fp_text user "${REFERENCE}"
-			(at 0 1.27 360)
+			(at 0 1.27 0)
 			(layer "F.Fab")
 			(effects
@@
 	)
 	(segment
+		(start 98.7531 121.45)
+		(end 99.7495 120.4536)
+		(width 0.762)
+		(layer "F.Cu")
+		(net 2)
+	)
+	(segment
 		(start 79.728 125.25)
 		(end 81.026 123.952)
@@
 	(segment
 		(start 98.3544 121.8487)
-		(end 99.7495 120.4536)
+		(end 98.75 121.4531)
 		(width 0.762)
 		(layer "F.Cu")
@@
 	)
 	(segment
+		(start 98.75 121.45)
+		(end 98.7531 121.45)
+		(width 0.762)
+		(layer "F.Cu")
+		(net 2)
+	)
+	(segment
 		(start 85 71)
 		(end 85 114.644)
@@
 	)
 	(segment
+		(start 98.75 121.4531)
+		(end 98.75 121.45)
+		(width 0.762)
+		(layer "F.Cu")
+		(net 2)
+	)
+	(segment
 		(start 74.551 127.381)
 		(end 74.551 126.199)
@@
 	)
 	(via
+		(at 98.75 121.45)
+		(size 0.6)
+		(drill 0.3)
+		(layers "F.Cu" "B.Cu")
+		(net 2)
+	)
+	(via
 		(at 102.7318 123.3169)
 		(size 0.7)
@@
 		(net 2)
 	)
+	(via
+		(at 103.85 123.15)
+		(size 0.6)
+		(drill 0.3)
+		(layers "F.Cu" "B.Cu")
+		(net 2)
+	)
+	(segment
+		(start 103.6 123.4)
+		(end 103.85 123.15)
+		(width 0.762)
+		(layer "B.Cu")
+		(net 2)
+	)
+	(segment
+		(start 102.7318 123.3169)
+		(end 102.8149 123.4)
+		(width 0.762)
+		(layer "B.Cu")
+		(net 2)
+	)
 	(segment
 		(start 102.6128 123.3169)
@@
 	)
 	(segment
+		(start 103.5 123.4)
+		(end 103.6 123.4)
+		(width 0.762)
+		(layer "B.Cu")
+		(net 2)
+	)
+	(segment
+		(start 103.85 123.15)
+		(end 103.881408 123.118592)
+		(width 0.762)
+		(layer "B.Cu")
+		(net 2)
+	)
+	(segment
+		(start 102.8149 123.4)
+		(end 103.5 123.4)
+		(width 0.762)
+		(layer "B.Cu")
+		(net 2)
+	)
+	(segment
+		(start 99.7495 120.4536)
+		(end 99.7464 120.4536)
+		(width 0.762)
+		(layer "B.Cu")
+		(net 2)
+	)
+	(segment
+		(start 99.7464 120.4536)
+		(end 98.755642 121.444358)
+		(width 0.762)
+		(layer "B.Cu")
+		(net 2)
+	)
+	(segment
 		(start 99.7495 120.4536)
 		(end 102.6128 123.3169)
@@
 	)
 	(segment
-		(start 91.8541 110.5)
-		(end 109.4127 128.0586)
+		(start 90.5 110.5)
+		(end 93.087804 110.5)
 		(width 0.3048)
 		(layer "B.Cu")
@@
 	)
 	(segment
-		(start 109.4127 128.0586)
+		(start 109.4127 126.824896)
 		(end 109.4127 128.5728)
 		(width 0.3048)
@@
 	)
 	(segment
-		(start 90.5 110.5)
-		(end 91.8541 110.5)
+		(start 93.087804 110.5)
+		(end 109.4127 126.824896)
 		(width 0.3048)
 		(layer "B.Cu")
@@
 	(segment
 		(start 90.5 113.04)
-		(end 91.8541 113.04)
+		(end 94.84 113.04)
 		(width 0.3048)
 		(layer "B.Cu")
@@
 	)
 	(segment
-		(start 93.4945 113.04)
-		(end 103.4669 123.0124)
-		(width 0.3048)
-		(layer "B.Cu")
-		(net 16)
-	)
-	(segment
-		(start 116.0336 132.0713)
-		(end 120.5723 136.61)
+		(start 94.84 113.04)
+		(end 105.15 123.35)
 		(width 0.3048)
 		(layer "B.Cu")
@@
 	)
 	(segment
-		(start 103.4669 123.578)
-		(end 111.9602 132.0713)
+		(start 120.5723 136.61)
+		(end 121.79 136.61)
 		(width 0.3048)
 		(layer "B.Cu")
@@
 	)
 	(segment
-		(start 121.79 136.61)
-		(end 120.5723 136.61)
+		(start 105.15 125.2611)
+		(end 111.9602 132.0713)
 		(width 0.3048)
 		(layer "B.Cu")
@@
 	)
 	(segment
-		(start 91.8541 113.04)
-		(end 93.4945 113.04)
+		(start 105.15 123.35)
+		(end 105.15 125.2611)
 		(width 0.3048)
 		(layer "B.Cu")
@@
 	)
 	(segment
-		(start 103.4669 123.0124)
-		(end 103.4669 123.578)
+		(start 116.0336 132.0713)
+		(end 120.5723 136.61)
 		(width 0.3048)
 		(layer "B.Cu")
